File: hw/kicad/smart_watch/smart_watch.kicad_sch (KiCad schematic)
At the start: 49 parts, among them J1 BATTERTY, J2 1051330001, J3 GC9A01, J4 JST_PH6, SW1 SW_Push, SW2 SW_Push, SW3 SW_Push, SW4 SW_Push, U1 STM32L476RGTx, U2 nPM1300-QEAA, U3 SHT41, U4 LIS2MDL, U5 CH340E, U6 DS3231MZ

Commit message: pcb design part 1
Parts:
- C20: footprint Capacitor_SMD:C_0201_0603Metric -> Capacitor_SMD:C_0603_1608Metric
- J3: footprint Connector_FFC-FPC:Molex_200528-0080_1x08-1MP_P1.00mm_Horizontal -> Connector_FFC-FPC:Hirose_FH12-15S-0.5SH_1x15-1MP_P0.50mm_Horizontal
- J4: value JST_PH6 -> JST_ZH6; footprint Connector_JST:JST_PH_S6B-PH-K_1x06_P2.00mm_Horizontal -> Connector_JST:JST_ZH_S6B-ZR-SM4A-TF_1x06-1MP_P1.50mm_Horizontal
Connections:
- net at D1.1: now also J2.2; no longer J2.3
- net at D1.3: now also J2.3; no longer J2.2
- net at D1.4: now also U5.1 (UD+); no longer U5.2 (UD-)
- net at D1.6: now also U5.2 (UD-); no longer U5.1 (UD+)
Other:
- note added: "NOTE: Molex 200528 8 pin FPC connector"
- note added: "NOTE: Molex PicoBlade 53261"
- note removed: "NOTE: 8 pin FPC connector"
Changed lines of the file:
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@@
 	(wire
 		(pts
-			(xy 229.87 147.32) (xy 238.76 147.32)
+			(xy 229.87 147.32) (xy 240.03 147.32)
 		)
 		(stroke
@@
 	(wire
 		(pts
+			(xy 238.76 132.08) (xy 238.76 139.7)
+		)
+		(stroke
+			(width 0)
+			(type default)
+		)
+	)
+	(wire
+		(pts
 			(xy 45.72 171.45) (xy 45.72 165.1)
 		)
@@
 	(wire
 		(pts
-			(xy 198.12 132.08) (xy 198.12 138.43)
-		)
-		(stroke
-			(width 0)
-			(type default)
-		)
-	)
-	(wire
-		(pts
 			(xy 115.57 71.12) (xy 121.92 71.12)
 		)
@@
 	(wire
 		(pts
-			(xy 194.31 147.32) (xy 204.47 147.32)
-		)
-		(stroke
-			(width 0)
-			(type default)
-		)
-	)
-	(wire
-		(pts
 			(xy 39.37 184.15) (xy 45.72 184.15)
 		)
@@
 	(wire
 		(pts
+			(xy 240.03 137.16) (xy 240.03 147.32)
+		)
+		(stroke
+			(width 0)
+			(type default)
+		)
+	)
+	(wire
+		(pts
 			(xy 207.01 33.02) (xy 214.63 33.02)
 		)
@@
 	(wire
 		(pts
+			(xy 198.12 138.43) (xy 198.12 147.32)
+		)
+		(stroke
+			(width 0)
+			(type default)
+		)
+	)
+	(wire
+		(pts
 			(xy 45.72 184.15) (xy 45.72 179.07)
 		)
@@
 	(wire
 		(pts
+			(xy 198.12 147.32) (xy 204.47 147.32)
+		)
+		(stroke
+			(width 0)
+			(type default)
+		)
+	)
+	(wire
+		(pts
 			(xy 129.54 125.73) (xy 133.35 125.73)
 		)
@@
 	(wire
 		(pts
-			(xy 187.96 135.89) (xy 194.31 135.89)
+			(xy 187.96 135.89) (xy 198.12 135.89)
 		)
 		(stroke
@@
 	(wire
 		(pts
-			(xy 194.31 135.89) (xy 194.31 147.32)
-		)
-		(stroke
-			(width 0)
-			(type default)
-		)
-	)
-	(wire
-		(pts
 			(xy 160.02 133.35) (xy 156.21 133.35)
 		)
@@
 	(wire
 		(pts
-			(xy 238.76 147.32) (xy 238.76 139.7)
-		)
-		(stroke
-			(width 0)
-			(type default)
-		)
-	)
-	(wire
-		(pts
 			(xy 105.41 74.93) (xy 105.41 78.74)
 		)
@@
 	(wire
 		(pts
-			(xy 238.76 132.08) (xy 238.76 137.16)
-		)
-		(stroke
-			(width 0)
-			(type default)
-		)
-	)
-	(wire
-		(pts
 			(xy 215.9 105.41) (xy 219.71 105.41)
 		)
@@
 	(wire
 		(pts
+			(xy 198.12 132.08) (xy 198.12 135.89)
+		)
+		(stroke
+			(width 0)
+			(type default)
+		)
+	)
+	(wire
+		(pts
 			(xy 158.75 177.8) (xy 161.29 177.8)
 		)
@@
 	(wire
 		(pts
-			(xy 238.76 137.16) (xy 247.65 137.16)
+			(xy 240.03 137.16) (xy 247.65 137.16)
 		)
 		(stroke
@@
 		)
 	)
+	(text "NOTE: \nMolex PicoBlade \n53261"
+		(exclude_from_sim no)
+		(at 95.25 38.354 0)
+		(effects
+			(font
+				(size 1.27 1.27)
+			)
+		)
+	)
 	(text "Temperature-Humidity Sensor"
 		(exclude_from_sim no)
@@
 		)
 	)
-	(text "NOTE: 8 pin FPC connector"
+	(text "NOTE: \nMolex 200528\n8 pin FPC connector"
 		(exclude_from_sim no)
-		(at 223.52 83.312 0)
+		(at 228.346 57.15 0)
 		(effects
 			(font
@@
 			)
 		)
-		(property "Footprint" "Connector_FFC-FPC:Molex_200528-0080_1x08-1MP_P1.00mm_Horizontal"
+		(property "Footprint" "Connector_FFC-FPC:Hirose_FH12-15S-0.5SH_1x15-1MP_P0.50mm_Horizontal"
 			(at 224.79 69.85 0)
 			(effects
@@
 			)
 		)
-		(property "Value" "JST_PH6"
+		(property "Value" "JST_ZH6"
 			(at 227.33 102.8699 0)
 			(effects
@@
 			)
 		)
-		(property "Footprint" "Connector_JST:JST_PH_S6B-PH-K_1x06_P2.00mm_Horizontal"
+		(property "Footprint" "Connector_JST:JST_ZH_S6B-ZR-SM4A-TF_1x06-1MP_P1.50mm_Horizontal"
 			(at 224.79 100.33 0)
 			(effects
@@
 			)
 		)
-		(property "Footprint" "Capacitor_SMD:C_0201_0603Metric"
+		(property "Footprint" "Capacitor_SMD:C_0603_1608Metric"
 			(at 112.7252 35.56 0)
 			(effects

Commit message: pcb design part 2
Parts:
- added C16: 100n, Capacitor_SMD:C_0603_1608Metric, symbol Device:C
Connections:
- net +3.3V: now also C16.1
- net GND: now also C16.2
Changed lines of the file:
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@@
 	)
 	(junction
+		(at 237.49 25.4)
+		(diameter 0)
+		(color 0 0 0 0)
+	)
+	(junction
 		(at 46.99 25.4)
 		(diameter 0)
@@
 	)
 	(junction
+		(at 237.49 33.02)
+		(diameter 0)
+		(color 0 0 0 0)
+	)
+	(junction
 		(at 39.37 184.15)
 		(diameter 0)
@@
 	(wire
 		(pts
+			(xy 237.49 33.02) (xy 245.11 33.02)
+		)
+		(stroke
+			(width 0)
+			(type default)
+		)
+	)
+	(wire
+		(pts
 			(xy 215.9 105.41) (xy 219.71 105.41)
 		)
@@
 	(wire
 		(pts
+			(xy 237.49 25.4) (xy 245.11 25.4)
+		)
+		(stroke
+			(width 0)
+			(type default)
+		)
+	)
+	(wire
+		(pts
 			(xy 195.58 128.27) (xy 195.58 133.35)
 		)
@@
 					(unit 1)
 				)
+			)
+		)
+	)
+	(symbol
+		(lib_id "Device:C")
+		(at 245.11 29.21 0)
+		(unit 1)
+		(exclude_from_sim no)
+		(in_bom yes)
+		(on_board yes)
+		(dnp no)
+		(property "Reference" "C16"
+			(at 245.872 26.924 0)
+			(effects
+				(font
+					(size 1.27 1.27)
+				)
+				(justify left)
+			)
+		)
+		(property "Value" "100n"
+			(at 245.872 31.496 0)
+			(effects
+				(font
+					(size 1.27 1.27)
+				)
+				(justify left)
+			)
+		)
+		(property "Footprint" "Capacitor_SMD:C_0603_1608Metric"
+			(at 246.0752 33.02 0)
+			(effects
+				(font
+					(size 1.27 1.27)
+				)
+				(hide yes)
+			)
+		)
+		(property "Datasheet" "~"
+			(at 245.11 29.21 0)
+			(effects
+				(font
+					(size 1.27 1.27)
+				)
+				(hide yes)
+			)
+		)
+		(property "Description" "Unpolarized capacitor"
+			(at 245.11 29.21 0)
+			(effects
+				(font
+					(size 1.27 1.27)
+				)
+				(hide yes)
+			)
+		)
+		(pin "1"
+		)
+		(pin "2"
+		)
+		(instances
+			(project "smart_watch"
+				(path "/4ac5f003-0b17-4e2a-b0b3-686063eb2ada"
+					(reference "C16")
+					(unit 1)
+				)

Commit message: layout attempt 2
Parts:
- removed C1: 100n, Capacitor_SMD:C_0603_1608Metric, symbol Device:C
- removed C51: 100u, Capacitor_SMD:C_0603_1608Metric, symbol Device:C
- removed J3: GC9A01, Connector_FFC-FPC:Hirose_FH12-15S-0.5SH_1x15-1MP_P0.50mm_Horizontal, symbol Connector_Generic:Conn_01x08
- removed J4: JST_ZH6, Connector_JST:JST_ZH_S6B-ZR-SM4A-TF_1x06-1MP_P1.50mm_Horizontal, symbol Connector_Generic:Conn_01x06
- removed R1: 10k, Resistor_SMD:R_0603_1608Metric, symbol Device:R
- added C2: 0.1u, Capacitor_SMD:C_0603_1608Metric, symbol Device:C
- added J3: GC9A01 / ER-TFT1.28-3, smart_watch:GC9A01_FPC_pads_P0.5mm, symbol Connector_Generic:Conn_01x15
- added J4: ZH7, Connector_JST:JST_ZH_S7B-ZR-SM4A-TF_1x07-1MP_P1.50mm_Horizontal, symbol Connector_Generic:Conn_01x07
Connections:
- net +3.3V: now also J3.4 (Pin_4), J4.1 (Pin_1); no longer SW1.1
- net BTN_2: now also U1.8 (PC0); no longer U1.26 (PB0)
- net GND: now also SW1.2, C2.1, J3.1 (Pin_1), J3.11 (Pin_11), J4.2 (Pin_2)
- net NRST: now also SW1.1, C2.2, J4.3 (Pin_3)
- net SPI_CS: now also J3.6 (Pin_6)
- net SPI_DC: now also J3.5 (Pin_5)
- net SPI_MOSI: now also J3.8 (Pin_8)
- net SPI_RST: now also J3.9 (Pin_9)
- net SPI_SCLK: now also J3.7 (Pin_7)
- net SWCLK: now also J4.6 (Pin_6)
- net SWDIO: now also J4.7 (Pin_7)
- net TDI: now reaches U1.50 (PA15)
- net TDI: now also J4.5 (Pin_5)
- net SWO: now reaches U1.55 (PB3)
- net SWO: now also J4.4 (Pin_4)
- removed net BTN_1: SW1.2, U1.8 (PC0)
- no-connect marks 56 -> 62
Other:
- note removed: "NOTE: Molex 200528 8 pin FPC connector"
- moved on the sheet: R11, SW1

Commit message: layout attempt 2 part 2
Connections:
- net +3.3V: now also J4.7 (Pin_7); no longer J4.1 (Pin_1)
- net GND: now also J4.6 (Pin_6); no longer J4.2 (Pin_2)
- net NRST: now also J4.5 (Pin_5); no longer J4.3 (Pin_3)
- net SWCLK: now also J4.2 (Pin_2); no longer J4.6 (Pin_6)
- net SWDIO: now also J4.1 (Pin_1); no longer J4.7 (Pin_7)
- net TDI: now also J4.3 (Pin_3); no longer J4.5 (Pin_5)

Commit message: Starting this again
Parts:
- removed U4: LIS2MDL, Package_LGA:LGA-12_2x2mm_P0.5mm, symbol Sensor_Magnetic:LIS2MDL
- added U4: ICM-20948, Sensor_Motion:InvenSense_QFN-24_3x3mm_P0.4mm, symbol Sensor_Motion:ICM-20948
- C40: value 10u -> 100n
- C42: value 220n -> 100n
Connections:
- net +1.8V: now also C40.2, C41.2, U4.13 (VDD), U4.8 (VDDIO); no longer C40.1, C41.1
- net GND: now also C40.1, C41.1, C42.1, U4.11 (FSYNC), U4.18 (GND), U4.20 (GND), U4.9 (SDO/AD0); no longer C40.2, C41.2, C42.2
- net I2C_SCL: now also U4.23 (SCL/SCLK)
- net I2C_SDA: now also U4.24 (SDA/SDI)
- net ICM_INT1: now reaches U1.59 (PB7)
- net ICM_INT1: now also U4.12 (INT1)
- new net: C42.2, U4.10 (REGOUT)
- no-connect marks 62 -> 63

Commit message: pcb design again pt 1
Parts:
- removed J3: GC9A01 / ER-TFT1.28-3, smart_watch:GC9A01_FPC_pads_P0.5mm, symbol Connector_Generic:Conn_01x15
- added J3: GC9A01 LCD, smart_watch:GC9A01_FPC_pads_P0.7mm, symbol Connector_Generic:Conn_01x12
- added Q1: 2N7000, Package_TO_SOT_SMD:SOT-23, symbol dk_Transistors-FETs-MOSFETs-Single:2N7000
- added R1: 0, Resistor_SMD:R_0603_1608Metric, symbol Device:R
Connections:
- net +3.3V: now also J3.3 (Pin_3), J3.4 (Pin_4)
- net GND: now also J3.1 (Pin_1), J3.12 (Pin_12), J3.5 (Pin_5), J3.6 (Pin_6), Q1.1 (S)
- net SPI_CS: now also J3.8 (Pin_8)
- net SPI_DC: now also J3.7 (Pin_7)
- net SPI_MOSI: now also J3.10 (Pin_10)
- net SPI_RST: now also J3.11 (Pin_11)
- net SPI_SCLK: now also J3.9 (Pin_9)
- net LCD_BKLGHT: now reaches U1.22 (PA6)
- net LCD_BKLGHT: now also Q1.2 (G)
- new net: Q1.3 (D), R1.1
- new net: J3.2 (Pin_2), R1.2
- no-connect marks 63 -> 55

Commit message: pcb design again pt 3
Connections:
- net BTN_2: now also U1.9 (PC1); no longer U1.8 (PC0)
- net BTN_4: now also U1.44 (PA11); no longer U1.53 (PC12)
- net ICM_INT1: now also U1.53 (PC12); no longer U1.59 (PB7)
- net LCD_BKLGHT: now also U1.16 (PA2); no longer U1.22 (PA6)
- net RTC_INT: now also U1.8 (PC0); no longer U1.52 (PC11)
- net SPI_CS: now also U1.28 (PB2); no longer U1.58 (PB6)
- net SPI_DC: now also U1.27 (PB1); no longer U1.43 (PA10)
- net SPI_RST: now also U1.30 (PB11); no longer U1.41 (PA8)
- net USART_RX: now also U1.25 (PC5); no longer U1.17 (PA3)
- net USART_TX: now also U1.24 (PC4); no longer U1.16 (PA2)
