File: hw/kicad/smart_watch/smart_watch.kicad_pcb (KiCad board)
At the start: 2 copper layers, 48 parts, among them J1 BATTERTY, J2 1051330001, J3 GC9A01 / ER-TFT1.28-3, J4 ZH7, SW1 SW_Push, SW2 SW_Push, SW3 SW_Push, SW4 SW_Push, U1 STM32L476RGTx, U2 nPM1300-QEAA, U3 SHT41, U4 ICM-20948, U5 CH340E, U6 DS3231MZ

Commit message: pcb design again pt 1
Parts:
- added Q1: 2N7000, Package_TO_SOT_SMD:SOT-23, F.Cu at (150.4, 122.7)
- added R1: 0, Resistor_SMD:R_0603_1608Metric, F.Cu at (152.6, 119.8)
- J1, J4: moved to B.Cu
- J3: value GC9A01 / ER-TFT1.28-3 -> GC9A01 LCD; footprint smart_watch:GC9A01_FPC_pads_P0.5mm -> smart_watch:GC9A01_FPC_pads_P0.7mm
- moved J1 154.3 mm to (96.2, 105.8), turned to 90 degrees
- moved SW2 131.6 mm to (120.7, 125.5)
- moved SW1 127.5 mm to (120.4, 85.5)
- moved U3 122.2 mm to (141.7, 89.4)
- moved J3 117.7 mm to (142.9, 122.8)
- moved U1 117.4 mm to (142.5, 111.3)
- moved R2 117.0 mm to (124.9, 125.5), turned to 180 degrees
- moved R5 114.8 mm to (128.7, 95.9), turned to 180 degrees
- moved C2 114.6 mm to (116.2, 85.5)
- moved C60 107.2 mm to (131.8, 95.9), turned to 180 degrees
- moved D1 107.1 mm to (155.8, 107.8)
- moved U4 104.3 mm to (137.5, 94.7)
- moved R12 104.3 mm to (139.2, 102.9), turned to 90 degrees
- moved U6 104.0 mm to (129.4, 100.5), turned to -90 degrees
- moved R11 103.0 mm to (140.8, 102.9), turned to -90 degrees
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Connections:
- J3 pad 10: unconnected-(J3-Pin_10-Pad10) -> /SPI_MOSI
- J3 pad 11: GND -> /SPI_RST
- J3 pad 12: unconnected-(J3-Pin_12-Pad12) -> GND
- J3 pad 2: unconnected-(J3-Pin_2-Pad2) -> Net-(J3-Pin_2)
- J3 pad 3: unconnected-(J3-Pin_3-Pad3) -> +3.3V
- J3 pad 5: /SPI_DC -> GND
- J3 pad 6: /SPI_CS -> GND
- J3 pad 7: /SPI_SCLK -> /SPI_DC
- J3 pad 8: /SPI_MOSI -> /SPI_CS
- J3 pad 9: /SPI_RST -> /SPI_SCLK
- U1 pad 22: unconnected-(U1-PA6-Pad22) -> /LCD_BKLGHT

Commit message: pcb design again pt 2
Parts:
- moved J4 54.0 mm to (208.1, 126.6), turned to 180 degrees
- moved J1 49.1 mm to (142.5, 89.5), turned to 0 degrees
- moved R1 17.2 mm to (135.4, 121.3)
- moved C2 16.5 mm to (128.5, 96.6)
- moved Q1 16.3 mm to (134.7, 118.3), turned to -90 degrees
- moved C60 15.9 mm to (126.3, 110.9), turned to 0 degrees
- moved R5 15.0 mm to (129.4, 110.9), turned to 0 degrees
- moved R4 15.0 mm to (156.4, 96.5)
- moved R3 14.8 mm to (152.2, 120.3), turned to 90 degrees
- moved SW1 12.3 mm to (129.8, 93.5), turned to 45 degrees
- moved SW2 11.2 mm to (129.8, 119.0), turned to 135 degrees
- moved SW4 10.7 mm to (155.2, 93.5), turned to -45 degrees
- moved R2 10.3 mm to (128.6, 115.9), turned to 0 degrees
- moved SW3 9.10 mm to (155.2, 119.0), turned to -135 degrees
- moved U3 6.34 mm to (136.4, 93.0)
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Routing:
- net /I2C_SDA: track 0.00 -> 34.0 mm, vias 0 -> 4
- net /I2C_SCL: track 0.00 -> 33.6 mm, vias 0 -> 4
- net +1.8V: track 0.00 -> 23.0 mm, vias 0 -> 4
- net +3.3V: track 0.00 -> 22.0 mm
- net /NRST: track 0.00 -> 20.8 mm
- net /VBUS: track 0.00 -> 17.0 mm, vias 0 -> 3
- net /VSYS: track 0.00 -> 15.8 mm, vias 0 -> 3
- net /BTN_2: track 0.00 -> 11.9 mm
- net Net-(D1-Pad1): track 0.00 -> 6.17 mm
- net Net-(J3-Pin_2): track 0.00 -> 5.09 mm
- net GND: track 0.00 -> 4.85 mm
- net Net-(D1-Pad3): track 0.00 -> 3.53 mm
- net Net-(U1-BOOT0): track 0.00 -> 2.92 mm
- net /RTC_INT: track 0.00 -> 2.54 mm
- net Net-(U2-VSET1): track 0.00 -> 2.47 mm
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Other:
- copper layers 2 -> 4

Commit message: pcb design again pt 3
Parts:
- moved J4 67.0 mm to (142.5, 113.0)
- moved D1 1.31 mm to (154.9, 105.8), turned to 90 degrees
- moved J3 0.70 mm to (142.5, 123.9)
- moved C13 0.30 mm to (139.1, 119.0)
- turned U5 to 180 degrees
Connections:
- U1 pad 16: /USART_TX -> /LCD_BKLGHT
- U1 pad 17: /USART_RX -> unconnected-(U1-PA3-Pad17)
- U1 pad 22: /LCD_BKLGHT -> unconnected-(U1-PA6-Pad22)
- U1 pad 24: unconnected-(U1-PC4-Pad24) -> /USART_TX
- U1 pad 25: unconnected-(U1-PC5-Pad25) -> /USART_RX
- U1 pad 27: unconnected-(U1-PB1-Pad27) -> /SPI_DC
- U1 pad 28: unconnected-(U1-PB2-Pad28) -> /SPI_CS
- U1 pad 30: unconnected-(U1-PB11-Pad30) -> /SPI_RST
- U1 pad 41: /SPI_RST -> unconnected-(U1-PA8-Pad41)
- U1 pad 43: /SPI_DC -> unconnected-(U1-PA10-Pad43)
- U1 pad 44: unconnected-(U1-PA11-Pad44) -> /BTN_4
- U1 pad 52: /RTC_INT -> unconnected-(U1-PC11-Pad52)
- U1 pad 53: /BTN_4 -> /ICM_INT1
- U1 pad 58: /SPI_CS -> unconnected-(U1-PB6-Pad58)
- U1 pad 59: /ICM_INT1 -> unconnected-(U1-PB7-Pad59)
- U1 pad 8: /BTN_2 -> /RTC_INT
- U1 pad 9: unconnected-(U1-PC1-Pad9) -> /BTN_2
Routing:
- net /NRST: track 20.8 -> 39.0 mm, vias 0 -> 3
- net /BTN_4: track 2.46 -> 20.2 mm
- net /USART_TX: track 0.00 -> 14.0 mm, vias 0 -> 2
- net Net-(J1-Pin_1): track 2.26 -> 15.8 mm, vias 0 -> 2
- net /ICM_INT1: track 0.00 -> 13.3 mm
- net /USART_RX: track 0.00 -> 13.3 mm, vias 0 -> 2
- net Net-(U5-UD+): track 0.00 -> 12.4 mm
- net /BTN_3: track 2.47 -> 12.5 mm
- net /I2C_SCL: track 33.6 -> 43.0 mm, vias 4 -> 5
- net Net-(U5-UD-): track 0.00 -> 9.31 mm, vias 0 -> 2
- net /SPI_SCLK: track 0.00 -> 7.67 mm
- net /SPI_MOSI: track 0.00 -> 7.55 mm
- net /SPI_DC: track 0.00 -> 7.25 mm, vias 0 -> 2
- net /SPI_CS: track 0.00 -> 7.21 mm, vias 0 -> 2
- net /I2C_SDA: track 34.0 -> 41.1 mm
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
Commit message: pcb design again pt 4
Parts:
- moved C42 1.12 mm to (135.6, 101.9), turned to 180 degrees
Connections:
- R11 pad 1: +3.3V -> GND
- R12 pad 2: +3.3V -> GND
Routing:
- net GND: track 4.85 -> 63.3 mm, vias 0 -> 48
- net +3.3V: track 22.4 -> 38.4 mm, vias 0 -> 19
- net +1.8V: track 23.0 -> 31.9 mm, vias 4 -> 5
- net /BTN_4: track 20.2 -> 20.9 mm
- net Net-(U4-REGOUT): track 1.47 -> 2.16 mm
- added copper zone on In2.Cu, net +3.3V
- added copper zone on In1.Cu, net GND
Other:
- board outline added: 40 x 40 mm
